File: hardware/storybox/storybox.kicad_pcb (KiCad board)
At the start: 2 copper layers, 62.7 x 82.1 mm, 22 parts, among them J3 Speaker, J4 Ext, J5 AudioJack, SW1 Prev, SW2 Next, SW3 Play, SW4 Home, U1 Pico, U2 Amplifier, U3 MicroSD Adafruit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

Commit message: inital  commut v3
Parts:
- added J1: Conn_01x01_Pin, Connector_PinHeader_2.54mm:PinHeader_1x01_P2.54mm_Vertical, F.Cu at (130.9, 116.3)
- added JP1: SolderJumper_2_Bridged, Jumper:SolderJumper-2_P1.3mm_Bridged_Pad1.0x1.5mm, F.Cu at (156.7, 65.9)
- added JP2: SolderJumper_2_Bridged, Jumper:SolderJumper-2_P1.3mm_Bridged_Pad1.0x1.5mm, F.Cu at (134.3, 116.3)
- added R3: 100k, Resistor_THT:R_Axial_DIN0204_L3.6mm_D1.6mm_P2.54mm_Vertical, F.Cu at (152.9, 66.9)
- D1: footprint Diode_THT:D_DO-34_SOD68_P7.62mm_Horizontal -> Diode_THT:D_DO-15_P10.16mm_Horizontal
- J4: moved to B.Cu
- On-Off1: value Switch -> SW_SPST
- moved J4 37.2 mm to (137.9, 75.9), turned to 180 degrees
- moved U5 8.99 mm to (169.6, 129.4)
- moved D1 2.16 mm to (153.0, 98.5)
- moved R2 2.16 mm to (157.7, 104.9)
- moved R1 2.16 mm to (157.6, 100.9)
- moved U2 1.31 mm to (142.2, 137.9)
Connections:
- J5 pad 4: Net-(J3-Pin_1) -> Net-(JP1-B)
- U1 pad 34: unconnected-(U1-GPIO28_ADC2-Pad34)_0 -> Net-(JP1-A)
- U2 pad 4: unconnected-(U2-Gain-Pad4) -> Net-(JP2-B)
- U2 pad 5: unconnected-(U2-SD-Pad5) -> Net-(J1-Pin_1)
- U2 pad 7: +5V -> +3V3
Routing:
- net GND: track 194.0 -> 0.00 mm
- net Net-(J3-Pin_2): track 107.8 -> 0.00 mm
- net Net-(U2-Speaker_+): track 105.1 -> 0.00 mm
- net +3V3: track 105.0 -> 0.00 mm
- net Net-(J3-Pin_1): track 79.6 -> 0.00 mm
- net +5V: track 63.0 -> 0.00 mm
- net Net-(J4-Pin_2): track 53.6 -> 0.00 mm
- net Net-(J4-Pin_4): track 53.1 -> 0.00 mm
- net Net-(J4-Pin_1): track 52.9 -> 0.00 mm, vias 1 -> 0
- net Net-(U1-GPIO16): track 47.6 -> 0.00 mm
- net Net-(J4-Pin_3): track 45.6 -> 0.00 mm
- net Net-(J4-Pin_6): track 44.7 -> 0.00 mm
- net Net-(D1-K): track 40.4 -> 0.00 mm
- net Net-(U1-GPIO22): track 39.0 -> 0.00 mm
- net Net-(J4-Pin_5): track 37.7 -> 0.00 mm
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- removed copper zone on B.Cu, net GND
- removed copper zone on F.Cu, net GND
Other:
- board text added: "Boite à histoire V3"
- board text added: "SW"
- board text removed: "3V"
- board text removed: "Boite à histoire V2"

Commit message: V3 pcb and latest code :-)
Parts:
- moved J4 0.23 mm to (137.8, 75.7)
Routing:
- net GND: track 0.00 -> 209.8 mm
- net +3V3: track 0.00 -> 110.3 mm, vias 0 -> 1
- net Net-(J3-Pin_2): track 0.00 -> 108.3 mm
- net Net-(U2-Speaker_+): track 0.00 -> 94.8 mm
- net Net-(D1-K): track 0.00 -> 76.2 mm
- net Net-(J3-Pin_1): track 0.00 -> 72.8 mm
- net +5V: track 0.00 -> 55.6 mm
- net Net-(U1-GPIO16): track 0.00 -> 40.5 mm
- net Net-(U1-GPIO18): track 0.00 -> 40.0 mm, vias 0 -> 1
- net Net-(U1-GPIO22): track 0.00 -> 38.9 mm
- net Net-(U1-GPIO27_ADC1): track 0.00 -> 37.4 mm
- net Net-(U1-GPIO20): track 0.00 -> 36.3 mm
- net Net-(U1-GPIO17): track 0.00 -> 34.6 mm
- net Net-(U1-GPIO13): track 0.00 -> 32.9 mm
- net Net-(On-Off1-A): track 0.00 -> 32.5 mm
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- added copper zone on B.Cu, net GND
- added copper zone on F.Cu, net GND
