File: hardware/storybox/storybox.kicad_sch (KiCad schematic)
At the start: 22 parts, among them J3 Speaker, J4 Ext, J5 AudioJack, SW1 Prev, SW2 Next, SW3 Play, SW4 Home, U1 Pico, U2 Amplifier, U3 MicroSD Adafruit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

Commit message: inital  commut v3
Parts:
- added J1: Conn_01x01_Pin, Connector_PinHeader_2.54mm:PinHeader_1x01_P2.54mm_Vertical, symbol Connector:Conn_01x01_Pin
- added JP1, JP2: SolderJumper_2_Bridged, Jumper:SolderJumper-2_P1.3mm_Bridged_Pad1.0x1.5mm, symbol Jumper:SolderJumper_2_Bridged
- added R3: 100k, Resistor_THT:R_Axial_DIN0204_L3.6mm_D1.6mm_P2.54mm_Vertical, symbol Device:R
- D1: footprint Diode_THT:D_DO-34_SOD68_P7.62mm_Horizontal -> Diode_THT:D_DO-15_P10.16mm_Horizontal
Connections:
- net +3V3: now also U2.7 (Vin), JP2.1 (A)
- net +5V: no longer U2.7 (Vin)
- net GND: now also R3.2
- net at J3.1 (Pin_1), J5.5: no longer J5.4
- net at U2.4 (Gain): now also JP2.2 (B)
- net at U2.5 (SD): now also J1.1 (Pin_1)
- net at U1.34 (GPIO28_ADC2): now also JP1.1 (A)
- new net: J5.4, JP1.2 (B), R3.1
- no-connect marks 25 -> 22
Other:
- moved on the sheet: J3
